Commit message: XML

File: robot_ws/src/myworkcell_support/urdf/robot.xacro (robot description, xacro)
@@ -156,5 +156,5 @@
   </collision>
 </link>
-<joint name="Rev3" type="continuous">
+<joint name="Rev1" type="continuous">
   <origin rpy="0 0 0" xyz="0.04741 0.151 0.0"/>
   <parent link="Component1_1"/>
@@ -163,15 +163,15 @@
   <limit effort="30" velocity="1.0" lower="-2" upper="1" />
 </joint>
-<transmission name="Rev3_tran">
-  <type>transmission_interface/SimpleTransmission</type>
-  <joint name="Rev3">
-    <hardwareInterface>PositionJointInterface</hardwareInterface>
-  </joint>
-  <actuator name="Rev3_actr">
-    <hardwareInterface>PositionJointInterface</hardwareInterface>
-    <mechanicalReduction>1</mechanicalReduction>
-  </actuator>
-</transmission>
-<joint name="Rev4" type="continuous">
+<transmission name="Rev1_tran">
+  <type>transmission_interface/SimpleTransmission</type>
+  <joint name="Rev1">
+    <hardwareInterface>PositionJointInterface</hardwareInterface>
+  </joint>
+  <actuator name="Rev1_actr">
+    <hardwareInterface>PositionJointInterface</hardwareInterface>
+    <mechanicalReduction>1</mechanicalReduction>
+  </actuator>
+</transmission>
+<joint name="Rev2" type="continuous">
   <origin rpy="0 0 0" xyz="-0.09391 0.46 0.0"/>
   <parent link="Component2_1"/>
@@ -179,15 +179,15 @@
   <axis xyz="-0.01 0.0 -0.0"/>
 </joint>
-<transmission name="Rev4_tran">
-  <type>transmission_interface/SimpleTransmission</type>
-  <joint name="Rev4">
-    <hardwareInterface>PositionJointInterface</hardwareInterface>
-  </joint>
-  <actuator name="Rev4_actr">
-    <hardwareInterface>PositionJointInterface</hardwareInterface>
-    <mechanicalReduction>1</mechanicalReduction>
-  </actuator>
-</transmission>
-<joint name="Rev5" type="continuous">
+<transmission name="Rev2_tran">
+  <type>transmission_interface/SimpleTransmission</type>
+  <joint name="Rev2">
+    <hardwareInterface>PositionJointInterface</hardwareInterface>
+  </joint>
+  <actuator name="Rev2_actr">
+    <hardwareInterface>PositionJointInterface</hardwareInterface>
+    <mechanicalReduction>1</mechanicalReduction>
+  </actuator>
+</transmission>
+<joint name="Rev3" type="continuous">
   <origin rpy="0 0 0" xyz="0.0465 0.106 0.015"/>
   <parent link="Component3_1"/>
@@ -195,15 +195,15 @@
   <axis xyz="-0.0 -0.0 0.01"/>
 </joint>
-<transmission name="Rev5_tran">
-  <type>transmission_interface/SimpleTransmission</type>
-  <joint name="Rev5">
-    <hardwareInterface>PositionJointInterface</hardwareInterface>
-  </joint>
-  <actuator name="Rev5_actr">
-    <hardwareInterface>PositionJointInterface</hardwareInterface>
-    <mechanicalReduction>1</mechanicalReduction>
-  </actuator>
-</transmission>
-<joint name="Rev6" type="continuous">
+<transmission name="Rev3_tran">
+  <type>transmission_interface/SimpleTransmission</type>
+  <joint name="Rev3">
+    <hardwareInterface>PositionJointInterface</hardwareInterface>
+  </joint>
+  <actuator name="Rev3_actr">
+    <hardwareInterface>PositionJointInterface</hardwareInterface>
+    <mechanicalReduction>1</mechanicalReduction>
+  </actuator>
+</transmission>
+<joint name="Rev4" type="continuous">
   <origin rpy="0 0 0" xyz="-0.04 0.0 0.481"/>
   <parent link="Component4_1"/>
@@ -211,15 +211,15 @@
   <axis xyz="-0.01 0.0 0.0"/>
 </joint>
-<transmission name="Rev6_tran">
-  <type>transmission_interface/SimpleTransmission</type>
-  <joint name="Rev6">
-    <hardwareInterface>PositionJointInterface</hardwareInterface>
-  </joint>
-  <actuator name="Rev6_actr">
-    <hardwareInterface>PositionJointInterface</hardwareInterface>
-    <mechanicalReduction>1</mechanicalReduction>
-  </actuator>
-</transmission>
-<joint name="Rev7" type="continuous">
+<transmission name="Rev4_tran">
+  <type>transmission_interface/SimpleTransmission</type>
+  <joint name="Rev4">
+    <hardwareInterface>PositionJointInterface</hardwareInterface>
+  </joint>
+  <actuator name="Rev4_actr">
+    <hardwareInterface>PositionJointInterface</hardwareInterface>
+    <mechanicalReduction>1</mechanicalReduction>
+  </actuator>
+</transmission>
+<joint name="Rev5" type="continuous">
   <origin rpy="0 0 0" xyz="0.04 0.0 0.052"/>
   <parent link="Component5_1"/>
@@ -227,15 +227,15 @@
   <axis xyz="0.0 -0.0 0.01"/>
 </joint>
-<transmission name="Rev7_tran">
-  <type>transmission_interface/SimpleTransmission</type>
-  <joint name="Rev7">
-    <hardwareInterface>PositionJointInterface</hardwareInterface>
-  </joint>
-  <actuator name="Rev7_actr">
-    <hardwareInterface>PositionJointInterface</hardwareInterface>
-    <mechanicalReduction>1</mechanicalReduction>
-  </actuator>
-</transmission>
-<joint name="Rev8" type="continuous">
+<transmission name="Rev5_tran">
+  <type>transmission_interface/SimpleTransmission</type>
+  <joint name="Rev5">
+    <hardwareInterface>PositionJointInterface</hardwareInterface>
+  </joint>
+  <actuator name="Rev5_actr">
+    <hardwareInterface>PositionJointInterface</hardwareInterface>
+    <mechanicalReduction>1</mechanicalReduction>
+  </actuator>
+</transmission>
+<joint name="Rev6" type="continuous">
   <origin rpy="0 0 0" xyz="0.2 -0.691257 0.0"/>
   <parent link="base_link"/>
@@ -243,10 +243,10 @@
   <axis xyz="0.0 0.01 0.0"/>
 </joint>
-<transmission name="Rev8_tran">
-  <type>transmission_interface/SimpleTransmission</type>
-  <joint name="Rev8">
-    <hardwareInterface>PositionJointInterface</hardwareInterface>
-  </joint>
-  <actuator name="Rev8_actr">
+<transmission name="Rev6_tran">
+  <type>transmission_interface/SimpleTransmission</type>
+  <joint name="Rev6">
+    <hardwareInterface>PositionJointInterface</hardwareInterface>
+  </joint>
+  <actuator name="Rev6_actr">
     <hardwareInterface>PositionJointInterface</hardwareInterface>
     <mechanicalReduction>1</mechanicalReduction>

Commit message: xacro

File: robot_ws/src/myworkcell_support/urdf/robot.xacro (robot description, xacro)
@@ -156,5 +156,5 @@
   </collision>
 </link>
-<joint name="Rev1" type="continuous">
+<joint name="Rev2" type="continuous">
   <origin rpy="0 0 0" xyz="0.04741 0.151 0.0"/>
   <parent link="Component1_1"/>
@@ -163,15 +163,15 @@
   <limit effort="30" velocity="1.0" lower="-2" upper="1" />
 </joint>
-<transmission name="Rev1_tran">
-  <type>transmission_interface/SimpleTransmission</type>
-  <joint name="Rev1">
-    <hardwareInterface>PositionJointInterface</hardwareInterface>
-  </joint>
-  <actuator name="Rev1_actr">
-    <hardwareInterface>PositionJointInterface</hardwareInterface>
-    <mechanicalReduction>1</mechanicalReduction>
-  </actuator>
-</transmission>
-<joint name="Rev2" type="continuous">
+<transmission name="Rev2_tran">
+  <type>transmission_interface/SimpleTransmission</type>
+  <joint name="Rev2">
+    <hardwareInterface>PositionJointInterface</hardwareInterface>
+  </joint>
+  <actuator name="Rev2_actr">
+    <hardwareInterface>PositionJointInterface</hardwareInterface>
+    <mechanicalReduction>1</mechanicalReduction>
+  </actuator>
+</transmission>
+<joint name="Rev3" type="continuous">
   <origin rpy="0 0 0" xyz="-0.09391 0.46 0.0"/>
   <parent link="Component2_1"/>
@@ -179,15 +179,15 @@
   <axis xyz="-0.01 0.0 -0.0"/>
 </joint>
-<transmission name="Rev2_tran">
-  <type>transmission_interface/SimpleTransmission</type>
-  <joint name="Rev2">
-    <hardwareInterface>PositionJointInterface</hardwareInterface>
-  </joint>
-  <actuator name="Rev2_actr">
-    <hardwareInterface>PositionJointInterface</hardwareInterface>
-    <mechanicalReduction>1</mechanicalReduction>
-  </actuator>
-</transmission>
-<joint name="Rev3" type="continuous">
+<transmission name="Rev3_tran">
+  <type>transmission_interface/SimpleTransmission</type>
+  <joint name="Rev3">
+    <hardwareInterface>PositionJointInterface</hardwareInterface>
+  </joint>
+  <actuator name="Rev3_actr">
+    <hardwareInterface>PositionJointInterface</hardwareInterface>
+    <mechanicalReduction>1</mechanicalReduction>
+  </actuator>
+</transmission>
+<joint name="Rev4" type="continuous">
   <origin rpy="0 0 0" xyz="0.0465 0.106 0.015"/>
   <parent link="Component3_1"/>
@@ -195,15 +195,15 @@
   <axis xyz="-0.0 -0.0 0.01"/>
 </joint>
-<transmission name="Rev3_tran">
-  <type>transmission_interface/SimpleTransmission</type>
-  <joint name="Rev3">
-    <hardwareInterface>PositionJointInterface</hardwareInterface>
-  </joint>
-  <actuator name="Rev3_actr">
-    <hardwareInterface>PositionJointInterface</hardwareInterface>
-    <mechanicalReduction>1</mechanicalReduction>
-  </actuator>
-</transmission>
-<joint name="Rev4" type="continuous">
+<transmission name="Rev4_tran">
+  <type>transmission_interface/SimpleTransmission</type>
+  <joint name="Rev4">
+    <hardwareInterface>PositionJointInterface</hardwareInterface>
+  </joint>
+  <actuator name="Rev4_actr">
+    <hardwareInterface>PositionJointInterface</hardwareInterface>
+    <mechanicalReduction>1</mechanicalReduction>
+  </actuator>
+</transmission>
+<joint name="Rev5" type="continuous">
   <origin rpy="0 0 0" xyz="-0.04 0.0 0.481"/>
   <parent link="Component4_1"/>
@@ -211,15 +211,15 @@
   <axis xyz="-0.01 0.0 0.0"/>
 </joint>
-<transmission name="Rev4_tran">
-  <type>transmission_interface/SimpleTransmission</type>
-  <joint name="Rev4">
-    <hardwareInterface>PositionJointInterface</hardwareInterface>
-  </joint>
-  <actuator name="Rev4_actr">
-    <hardwareInterface>PositionJointInterface</hardwareInterface>
-    <mechanicalReduction>1</mechanicalReduction>
-  </actuator>
-</transmission>
-<joint name="Rev5" type="continuous">
+<transmission name="Rev5_tran">
+  <type>transmission_interface/SimpleTransmission</type>
+  <joint name="Rev5">
+    <hardwareInterface>PositionJointInterface</hardwareInterface>
+  </joint>
+  <actuator name="Rev5_actr">
+    <hardwareInterface>PositionJointInterface</hardwareInterface>
+    <mechanicalReduction>1</mechanicalReduction>
+  </actuator>
+</transmission>
+<joint name="Rev6" type="continuous">
   <origin rpy="0 0 0" xyz="0.04 0.0 0.052"/>
   <parent link="Component5_1"/>
@@ -227,15 +227,15 @@
   <axis xyz="0.0 -0.0 0.01"/>
 </joint>
-<transmission name="Rev5_tran">
-  <type>transmission_interface/SimpleTransmission</type>
-  <joint name="Rev5">
-    <hardwareInterface>PositionJointInterface</hardwareInterface>
-  </joint>
-  <actuator name="Rev5_actr">
-    <hardwareInterface>PositionJointInterface</hardwareInterface>
-    <mechanicalReduction>1</mechanicalReduction>
-  </actuator>
-</transmission>
-<joint name="Rev6" type="continuous">
+<transmission name="Rev6_tran">
+  <type>transmission_interface/SimpleTransmission</type>
+  <joint name="Rev6">
+    <hardwareInterface>PositionJointInterface</hardwareInterface>
+  </joint>
+  <actuator name="Rev6_actr">
+    <hardwareInterface>PositionJointInterface</hardwareInterface>
+    <mechanicalReduction>1</mechanicalReduction>
+  </actuator>
+</transmission>
+<joint name="Rev1" type="continuous">
   <origin rpy="0 0 0" xyz="0.2 -0.691257 0.0"/>
   <parent link="base_link"/>
@@ -243,10 +243,10 @@
   <axis xyz="0.0 0.01 0.0"/>
 </joint>
-<transmission name="Rev6_tran">
-  <type>transmission_interface/SimpleTransmission</type>
-  <joint name="Rev6">
-    <hardwareInterface>PositionJointInterface</hardwareInterface>
-  </joint>
-  <actuator name="Rev6_actr">
+<transmission name="Rev1_tran">
+  <type>transmission_interface/SimpleTransmission</type>
+  <joint name="Rev1">
+    <hardwareInterface>PositionJointInterface</hardwareInterface>
+  </joint>
+  <actuator name="Rev1_actr">
     <hardwareInterface>PositionJointInterface</hardwareInterface>
     <mechanicalReduction>1</mechanicalReduction>

Commit message: driver_node

File: robot_ws/src/myworkcell_support/urdf/robot.xacro (robot description, xacro)
@@ -178,4 +178,5 @@
   <child link="Component3_1"/>
   <axis xyz="-0.01 0.0 -0.0"/>
+  <limit effort="30" velocity="1.0" lower="-2.2" upper="0.7" />
 </joint>
 <transmission name="Rev3_tran">
