Commit message: urdf

File: robot_ws/src/nsra_support/urdf/robot.xacro (robot description, xacro)
@@ -11,5 +11,5 @@
     <origin rpy="0 0 0" xyz="0 0 0"/>
     <geometry>
-      <mesh filename="package://myworkcell_support/urdf/mm_stl/base_link.stl" scale="0.001 0.001 0.001"/>
+      <mesh filename="package://nsra_support/urdf/mm_stl/base_link.stl" scale="0.001 0.001 0.001"/>
     </geometry>
     <material name="silver">
@@ -20,5 +20,5 @@
     <origin rpy="0 0 0" xyz="0 0 0"/>
     <geometry>
-      <mesh filename="package://myworkcell_support/urdf/mm_stl/base_link.stl" scale="0.001 0.001 0.001"/>
+      <mesh filename="package://nsra_support/urdf/mm_stl/base_link.stl" scale="0.001 0.001 0.001"/>
     </geometry>
   </collision>
@@ -33,5 +33,5 @@
     <origin rpy="0 0 0" xyz="-0.24741 0.540257 -0.0"/>
     <geometry>
-      <mesh filename="package://myworkcell_support/urdf/mm_stl/Component2_1.stl" scale="0.001 0.001 0.001"/>
+      <mesh filename="package://nsra_support/urdf/mm_stl/Component2_1.stl" scale="0.001 0.001 0.001"/>
     </geometry>
     <material name="silver">
@@ -42,5 +42,5 @@
     <origin rpy="0 0 0" xyz="-0.24741 0.540257 -0.0"/>
     <geometry>
-      <mesh filename="package://myworkcell_support/urdf/mm_stl/Component2_1.stl" scale="0.001 0.001 0.001"/>
+      <mesh filename="package://nsra_support/urdf/mm_stl/Component2_1.stl" scale="0.001 0.001 0.001"/>
     </geometry>
   </collision>
@@ -55,5 +55,5 @@
     <origin rpy="0 0 0" xyz="-0.1535 0.080257 -0.0"/>
     <geometry>
-      <mesh filename="package://myworkcell_support/urdf/mm_stl/Component3_1.stl" scale="0.001 0.001 0.001"/>
+      <mesh filename="package://nsra_support/urdf/mm_stl/Component3_1.stl" scale="0.001 0.001 0.001"/>
     </geometry>
     <material name="silver">
@@ -64,5 +64,5 @@
     <origin rpy="0 0 0" xyz="-0.1535 0.080257 -0.0"/>
     <geometry>
-      <mesh filename="package://myworkcell_support/urdf/mm_stl/Component3_1.stl" scale="0.001 0.001 0.001"/>
+      <mesh filename="package://nsra_support/urdf/mm_stl/Component3_1.stl" scale="0.001 0.001 0.001"/>
     </geometry>
   </collision>
@@ -77,5 +77,5 @@
     <origin rpy="0 0 0" xyz="-0.2 -0.025743 -0.015"/>
     <geometry>
-      <mesh filename="package://myworkcell_support/urdf/mm_stl/Component4_1.stl" scale="0.001 0.001 0.001"/>
+      <mesh filename="package://nsra_support/urdf/mm_stl/Component4_1.stl" scale="0.001 0.001 0.001"/>
     </geometry>
     <material name="silver">
@@ -86,5 +86,5 @@
     <origin rpy="0 0 0" xyz="-0.2 -0.025743 -0.015"/>
     <geometry>
-      <mesh filename="package://myworkcell_support/urdf/mm_stl/Component4_1.stl" scale="0.001 0.001 0.001"/>
+      <mesh filename="package://nsra_support/urdf/mm_stl/Component4_1.stl" scale="0.001 0.001 0.001"/>
     </geometry>
   </collision>
@@ -99,5 +99,5 @@
     <origin rpy="0 0 0" xyz="-0.16 -0.025743 -0.496"/>
     <geometry>
-      <mesh filename="package://myworkcell_support/urdf/mm_stl/Component5_1.stl" scale="0.001 0.001 0.001"/>
+      <mesh filename="package://nsra_support/urdf/mm_stl/Component5_1.stl" scale="0.001 0.001 0.001"/>
     </geometry>
     <material name="silver">
@@ -108,5 +108,5 @@
     <origin rpy="0 0 0" xyz="-0.16 -0.025743 -0.496"/>
     <geometry>
-      <mesh filename="package://myworkcell_support/urdf/mm_stl/Component5_1.stl" scale="0.001 0.001 0.001"/>
+      <mesh filename="package://nsra_support/urdf/mm_stl/Component5_1.stl" scale="0.001 0.001 0.001"/>
     </geometry>
   </collision>
@@ -121,5 +121,5 @@
     <origin rpy="0 0 0" xyz="-0.2 -0.025743 -0.548"/>
     <geometry>
-      <mesh filename="package://myworkcell_support/urdf/mm_stl/Component6_1.stl" scale="0.001 0.001 0.001"/>
+      <mesh filename="package://nsra_support/urdf/mm_stl/Component6_1.stl" scale="0.001 0.001 0.001"/>
     </geometry>
     <material name="silver">
@@ -130,5 +130,5 @@
     <origin rpy="0 0 0" xyz="-0.2 -0.025743 -0.548"/>
     <geometry>
-      <mesh filename="package://myworkcell_support/urdf/mm_stl/Component6_1.stl" scale="0.001 0.001 0.001"/>
+      <mesh filename="package://nsra_support/urdf/mm_stl/Component6_1.stl" scale="0.001 0.001 0.001"/>
     </geometry>
   </collision>
@@ -143,5 +143,5 @@
     <origin rpy="0 0 0" xyz="-0.2 0.691257 0.0"/>
     <geometry>
-      <mesh filename="package://myworkcell_support/urdf/mm_stl/Component1_1.stl" scale="0.001 0.001 0.001"/>
+      <mesh filename="package://nsra_support/urdf/mm_stl/Component1_1.stl" scale="0.001 0.001 0.001"/>
     </geometry>
     <material name="silver">
@@ -152,5 +152,5 @@
     <origin rpy="0 0 0" xyz="-0.2 0.691257 0.0"/>
     <geometry>
-      <mesh filename="package://myworkcell_support/urdf/mm_stl/Component1_1.stl" scale="0.001 0.001 0.001"/>
+      <mesh filename="package://nsra_support/urdf/mm_stl/Component1_1.stl" scale="0.001 0.001 0.001"/>
     </geometry>
   </collision>
